Commit message: new branch

File: realsense2_description/urdf/_d435.urdf.xacro (robot description, xacro)
@@ -12,4 +12,5 @@
   <xacro:include filename="$(find realsense2_description)/urdf/_d435.gazebo.xacro"/>
   <xacro:macro name="sensor_d435" params="parent *origin name:=camera use_nominal_extrinsics:=false add_plug:=false use_mesh:=true">
+  <!-- <xacro:macro name="sensor_d435" params="name:=camera use_nominal_extrinsics:=false add_plug:=false use_mesh:=true"> -->
     <xacro:property name="M_PI" value="3.1415926535897931" />
     <!-- The following values are approximate, and the camera node

File: realsense2_description/urdf/test_d435_camera.urdf.xacro (robot description, xacro)
@@ -5,7 +5,5 @@
   <xacro:arg name="use_mesh" default="true" />
   <xacro:include filename="$(find realsense2_description)/urdf/_d435.urdf.xacro" />
-  <link name="base_link" />
-  <xacro:sensor_d435 parent="base_link" use_nominal_extrinsics="$(arg use_nominal_extrinsics)" add_plug="$(arg add_plug)" use_mesh="$(arg use_mesh)">
-    <origin xyz="0 0 0" rpy="0 0 0"/>
+  <xacro:sensor_d435 use_nominal_extrinsics="$(arg use_nominal_extrinsics)" add_plug="$(arg add_plug)" use_mesh="$(arg use_mesh)">
   </xacro:sensor_d435>
 </robot>

Commit message: collision and point cloud stream fixing

File: realsense2_description/urdf/_d435.urdf.xacro (robot description, xacro)
@@ -66,5 +66,5 @@
         </xacro:unless>
       </visual>
-      <collision>
+      <!-- <collision>
         <origin xyz="-0.0085 ${-d435_cam_depth_py} 0" rpy="0 0 0"/>
         <geometry>
